Commit message: v4

File: urdf/export.urdf (robot description, URDF)
Before this commit: robot export_test, 13 links, 12 joints
Joints:
- joint joint_left_ankle_pitch: limit lower=-0.6981 upper=0.6981 effort=500 velocity=1 -> lower=-0.6981 upper=0.6981 effort=1000 velocity=10
- joint joint_left_ankle_roll: limit lower=-0.5236 upper=0.5236 effort=500 velocity=1 -> lower=-0.5236 upper=0.5236 effort=1000 velocity=10
- joint joint_left_hip_pitch: limit lower=-0.1745 upper=1.5 effort=500 velocity=1 -> lower=-0.1745 upper=1.5 effort=1000 velocity=10
- joint joint_left_hip_roll: limit lower=-0.3108 upper=0.3108 effort=500 velocity=1 -> lower=-0.3108 upper=0.3108 effort=1000 velocity=10
- joint joint_left_hip_yaw: limit lower=-0.6 upper=0.2 effort=500 velocity=1 -> lower=-0.6 upper=0.2 effort=1000 velocity=10; origin xyz=0.139999999999999 0 0.0538 rpy=-3.14 0 0 -> xyz=-0 0.14 0.0538 rpy=-3.14 0 1.5708
- joint joint_left_knee_pitch: limit lower=-2.617 upper=0 effort=500 velocity=1 -> lower=-2.617 upper=0 effort=1000 velocity=10
- joint joint_right_ankle_pitch: limit lower=-0.6981 upper=0.6981 effort=500 velocity=1 -> lower=-0.6981 upper=0.6981 effort=1000 velocity=10
- joint joint_right_ankle_roll: limit lower=-0.5236 upper=0.5236 effort=500 velocity=1 -> lower=-0.5236 upper=0.5236 effort=1000 velocity=10
- joint joint_right_hip_pitch: limit lower=-0.1745 upper=1.5 effort=500 velocity=1 -> lower=-0.1745 upper=1.5 effort=1000 velocity=10
- joint joint_right_hip_roll: limit lower=-0.3108 upper=0.3108 effort=500 velocity=1 -> lower=-0.3108 upper=0.3108 effort=1000 velocity=10
- joint joint_right_hip_yaw: limit lower=-0.2 upper=0.6 effort=500 velocity=1 -> lower=-0.2 upper=0.6 effort=1000 velocity=10; origin xyz=-0.139999999999999 0 0.0538 rpy=-3.14 0 0 -> xyz=-0 -0.14 0.0538 rpy=-3.14 0 1.5708
- joint joint_right_knee_pitch: limit lower=0 upper=2.617 effort=500 velocity=1 -> lower=0 upper=2.617 effort=1000 velocity=10

Commit message: collision

File: urdf/export.urdf (robot description, URDF)
Before this commit: robot export_test, 13 links, 12 joints
Links:
- link base_link: geometry collision box size=0.10 0.08 0.05; visual mesh filename=../meshes/base_waist.obj
- link link_left_ankle_pitch: geometry visual mesh filename=../meshes/link_left_ankle_pitch.obj
- link link_left_hip_roll: geometry collision sphere radius=0.05; visual mesh filename=../meshes/link_left_hip_roll.obj
- link link_left_hip_yaw: geometry collision sphere radius=0.05; visual mesh filename=../meshes/link_left_hip_yaw.obj
- link link_left_shank: geometry collision cylinder length=0.2 radius=0.025; visual mesh filename=../meshes/link_left_shank.obj
- link link_left_thigh: geometry collision cylinder length=0.2 radius=0.045; visual mesh filename=../meshes/link_left_thigh.obj
- link link_right_ankle_pitch: geometry visual mesh filename=../meshes/link_right_ankle_pitch.obj
- link link_right_hip_roll: geometry collision sphere radius=0.05; visual mesh filename=../meshes/link_right_hip_roll.obj
- link link_right_hip_yaw: geometry collision sphere radius=0.05; visual mesh filename=../meshes/link_right_hip_yaw.obj
- link link_right_shank: geometry collision cylinder length=0.2 radius=0.025; visual mesh filename=../meshes/link_right_shank.obj
- link link_right_thigh: geometry collision cylinder length=0.2 radius=0.045; visual mesh filename=../meshes/link_right_thigh.obj

Commit message: collision1

File: urdf/export.urdf (robot description, URDF)
Before this commit: robot export_test, 13 links, 12 joints
Links:
- link link_left_ankle_roll: geometry collision box size=0.05 0.01 0.25; visual mesh filename=../meshes/link_left_ankle_roll.obj
- link link_right_ankle_roll: geometry collision box size=0.05 0.01 0.25; visual mesh filename=../meshes/link_right_ankle_roll.obj

Commit message: 足底碰撞修复

File: urdf/export.urdf (robot description, URDF)
Before this commit: robot export_test, 13 links, 12 joints
Links:
- link link_left_ankle_roll: geometry collision mesh filename=../meshes/link_left_ankle_roll.obj; visual mesh filename=../meshes/link_left_ankle_roll.obj
- link link_right_ankle_roll: geometry collision mesh filename=../meshes/link_right_ankle_roll.obj; visual mesh filename=../meshes/link_right_ankle_roll.obj

Commit message: baselink recover

File: urdf/export.urdf (robot description, URDF)
Before this commit: robot export_test, 13 links, 12 joints
Joints:
- joint joint_left_ankle_pitch: limit lower=-0.6981 upper=0.6981 effort=1000 velocity=10 -> lower=-0.6 upper=0.6 effort=1000 velocity=10; origin xyz=5.8589224897293E-05 -0.354999995165215 0 rpy=0 0 3.14 -> xyz=0 -0.3549 0 rpy=0 0 3.14
- joint joint_left_ankle_roll: axis 0 -0.00016500720596889 0.999999986386311 -> 0 0 1; limit lower=-0.5236 upper=0.5236 effort=1000 velocity=10 -> lower=-0.52 upper=0.52 effort=1000 velocity=10
- joint joint_left_hip_pitch: axis 0 0 -1 -> 0 0 1; limit lower=-0.1745 upper=1.5 effort=1000 velocity=10 -> lower=-1.5 upper=0.3 effort=1000 velocity=10
- joint joint_left_hip_roll: limit lower=-0.3108 upper=0.3108 effort=1000 velocity=10 -> lower=-0.15 upper=0.15 effort=1000 velocity=10
- joint joint_left_hip_yaw: limit lower=-0.6 upper=0.2 effort=1000 velocity=10 -> lower=-0.6 upper=0.4 effort=1000 velocity=10; origin xyz=-0 0.14 0.0538 rpy=-3.14 0 1.5708 -> xyz=0.13999 0 0.0538 rpy=-3.14 0 0
- joint joint_left_knee_pitch: limit lower=-2.617 upper=0 effort=1000 velocity=10 -> lower=-2.2 upper=0 effort=1000 velocity=10; origin xyz=-4.45034871792752E-05 -0.385203966374574 -0.0144999999997881 rpy=0 0 0 -> xyz=0 -0.3852 -0.0144 rpy=0 0 0
- joint joint_right_ankle_pitch: axis 0 0 -1 -> 0 0 1; limit lower=-0.6981 upper=0.6981 effort=1000 velocity=10 -> lower=-0.6 upper=0.6 effort=1000 velocity=10; origin xyz=0.355 5.8589E-05 0 rpy=0 0 4.71 -> xyz=0.355 0 0 rpy=0 0 4.71
- joint joint_right_ankle_roll: axis 0 -0.00016501 1 -> 0 0 1; limit lower=-0.5236 upper=0.5236 effort=1000 velocity=10 -> lower=-0.52 upper=0.52 effort=1000 velocity=10
- joint joint_right_hip_pitch: axis 0 0 -1 -> 0 0 1; limit lower=-0.1745 upper=1.5 effort=1000 velocity=10 -> lower=-1.5 upper=0.3 effort=1000 velocity=10
- joint joint_right_hip_roll: axis 0 0 -1 -> 0 0 1; limit lower=-0.3108 upper=0.3108 effort=1000 velocity=10 -> lower=-0.15 upper=0.15 effort=1000 velocity=10
- joint joint_right_hip_yaw: axis 0 0 -1 -> 0 0 1; limit lower=-0.2 upper=0.6 effort=1000 velocity=10 -> lower=-0.6 upper=0.4 effort=1000 velocity=10; origin xyz=-0 -0.14 0.0538 rpy=-3.14 0 1.5708 -> xyz=-0.13999 0 0.0538 rpy=-3.14 0 0
- joint joint_right_knee_pitch: axis 0 0 1 -> 0 0 -1; limit lower=0 upper=2.617 effort=1000 velocity=10 -> lower=-2.2 upper=0 effort=1000 velocity=10; origin xyz=-4.45034871116084E-05 -0.38520396637472 0.0254999999997153 rpy=0 0 -1.5707963267949 -> xyz=0 -0.38520 0.0254 rpy=0 0 -1.5707
