Commit message: Update BSRL URDF assets

File: urdf/export.urdf (robot description, URDF)
Before this commit: robot export_test, 13 links, 12 joints
Links:
- link base_link: geometry collision box size=0.08 0.1 0.05; visual mesh filename=../meshes/base_waist.obj
- link link_left_ankle_roll: geometry collision box size=0.25249708 0.08 0.10002095; visual mesh filename=../meshes/link_left_ankle_roll.obj
- link link_right_ankle_roll: geometry collision box size=0.25249708 0.08 0.10002095; visual mesh filename=../meshes/link_right_ankle_roll.obj
Joints:
- joint joint_left_ankle_pitch: axis 0 0 1 -> 0 1 0; origin xyz=0 -0.3549 0 rpy=0 0 3.14 -> xyz=0 0 -0.3549 rpy=0 0 0
- joint joint_left_ankle_roll: axis 0 0 1 -> 1 0 0; origin xyz=0 0 0 rpy=3.1415 -1.57 0 -> xyz=0 0 0 rpy=0 0 0
- joint joint_left_hip_pitch: axis 0 0 1 -> 0 1 0; origin xyz=0 0 0.104999999999906 rpy=0 1.5707963267949 0 -> xyz=0.105 0 0 rpy=0 0 0
- joint joint_left_hip_roll: axis 0 0 -1 -> -1 0 0; origin xyz=-0.000499999999956591 -0.102999999999988 0.110799999999914 rpy=-1.5707963267949 0 0 -> xyz=-0.103 -0.000499999999957 -0.1108 rpy=0 0 0
- joint joint_left_hip_yaw: axis 0 0 -1 -> 0 0 1; origin xyz=0.13999 0 0.0538 rpy=-3.14 0 0 -> xyz=0 0.13999 0.0538 rpy=0 0 0
- joint joint_left_knee_pitch: axis 0 0 -1 -> 0 -1 0; origin xyz=0 -0.3852 -0.0144 rpy=0 0 0 -> xyz=0 -0.0144 -0.3852 rpy=0 0 0
- joint joint_right_ankle_pitch: axis 0 0 1 -> 0 1 0; origin xyz=0.355 0 0 rpy=0 0 4.71 -> xyz=0 0 -0.355 rpy=0 0 0
- joint joint_right_ankle_roll: axis 0 0 1 -> 1 0 0; origin xyz=0 0 0 rpy=3.1416 -1.5708 0 -> xyz=0 0 0 rpy=0 0 0
- joint joint_right_hip_pitch: axis 0 0 1 -> 0 1 0; origin xyz=-0.0109999999999572 0 0.104999999999975 rpy=0 1.5707963267949 0 -> xyz=0.105 -0.011 0 rpy=0 0 0
- joint joint_right_hip_roll: axis 0 0 1 -> 1 0 0; origin xyz=0.0005 -0.103 0.1108 rpy=-1.5708 0 0 -> xyz=-0.103 0.0005 -0.1108 rpy=0 0 0
- joint joint_right_hip_yaw: axis 0 0 1 -> 0 0 -1; origin xyz=-0.13999 0 0.0538 rpy=-3.14 0 0 -> xyz=0 -0.13999 0.0538 rpy=0 0 0
- joint joint_right_knee_pitch: axis 0 0 -1 -> 0 -1 0; origin xyz=0 -0.38520 0.0254 rpy=0 0 -1.5707 -> xyz=0 0.0254 -0.3852 rpy=0 0 0

Commit message: inertia and mass update

File: urdf/export.urdf (robot description, URDF)
Before this commit: robot export, 13 links, 12 joints
Links:
- link base_link: mass 4.0754 -> 4.027447
- link link_left_ankle_pitch: mass 0.0552295043338537 -> 0.091152
- link link_left_ankle_roll: mass 1.29532298157718 -> 0.831234
- link link_left_hip_roll: mass 0.405320507205102 -> 1.620465
- link link_left_hip_yaw: mass 0.510408958903103 -> 1.725555
- link link_left_shank: mass 2.25275396724244 -> 2.492309
- link link_left_thigh: mass 1.38692340907035 -> 2.542662
- link link_right_ankle_pitch: mass 0.0552295043338538 -> 0.091152
- link link_right_ankle_roll: mass 1.29449582402577 -> 0.831235
- link link_right_hip_roll: mass 0.40532048161893 -> 1.620465
- link link_right_hip_yaw: mass 0.510408958903103 -> 1.725554
- link link_right_shank: mass 2.25642912872179 -> 2.492287
- link link_right_thigh: mass 1.38659078423411 -> 2.556965

Commit message: Unify BSRL joint axes and limits

File: urdf/export.urdf (robot description, URDF)
Before this commit: robot export, 13 links, 12 joints
Joints:
- joint joint_left_hip_roll: axis -1 0 0 -> 1 0 0
- joint joint_left_knee_pitch: axis 0 -1 0 -> 0 1 0; limit lower=-2.2 upper=0 effort=1000 velocity=10 -> lower=0 upper=2.2 effort=1000 velocity=10
- joint joint_right_hip_yaw: axis 0 0 -1 -> 0 0 1; limit lower=-0.6 upper=0.4 effort=1000 velocity=10 -> lower=-0.4 upper=0.6 effort=1000 velocity=10
- joint joint_right_knee_pitch: axis 0 -1 0 -> 0 1 0; limit lower=-2.2 upper=0 effort=1000 velocity=10 -> lower=0 upper=2.2 effort=1000 velocity=10

Commit message: Update BSRL motor limits in robot assets

File: urdf/export.urdf (robot description, URDF)
Before this commit: robot export, 13 links, 12 joints
Joints:
- joint joint_left_ankle_pitch: limit lower=-0.6 upper=0.6 effort=1000 velocity=10 -> lower=-0.6 upper=0.6 effort=112 velocity=26.1799
- joint joint_left_ankle_roll: limit lower=-0.52 upper=0.52 effort=1000 velocity=10 -> lower=-0.52 upper=0.52 effort=112 velocity=26.1799
- joint joint_left_hip_pitch: limit lower=-1.5 upper=0.3 effort=1000 velocity=10 -> lower=-1.5 upper=0.3 effort=216 velocity=15.1320
- joint joint_left_hip_roll: limit lower=-0.15 upper=0.15 effort=1000 velocity=10 -> lower=-0.15 upper=0.15 effort=216 velocity=15.1320
- joint joint_left_hip_yaw: limit lower=-0.6 upper=0.4 effort=1000 velocity=10 -> lower=-0.6 upper=0.4 effort=112 velocity=26.1799
- joint joint_left_knee_pitch: limit lower=0 upper=2.2 effort=1000 velocity=10 -> lower=0 upper=2.2 effort=216 velocity=15.1320
- joint joint_right_ankle_pitch: limit lower=-0.6 upper=0.6 effort=1000 velocity=10 -> lower=-0.6 upper=0.6 effort=112 velocity=26.1799
- joint joint_right_ankle_roll: limit lower=-0.52 upper=0.52 effort=1000 velocity=10 -> lower=-0.52 upper=0.52 effort=112 velocity=26.1799
- joint joint_right_hip_pitch: limit lower=-1.5 upper=0.3 effort=1000 velocity=10 -> lower=-1.5 upper=0.3 effort=216 velocity=15.1320
- joint joint_right_hip_roll: limit lower=-0.15 upper=0.15 effort=1000 velocity=10 -> lower=-0.15 upper=0.15 effort=216 velocity=15.1320
- joint joint_right_hip_yaw: limit lower=-0.4 upper=0.6 effort=1000 velocity=10 -> lower=-0.4 upper=0.6 effort=112 velocity=26.1799
- joint joint_right_knee_pitch: limit lower=0 upper=2.2 effort=1000 velocity=10 -> lower=0 upper=2.2 effort=216 velocity=15.1320

File: urdf/export_floating.urdf (robot description, URDF)
Before this commit: robot export_floating, 14 links, 13 joints
Joints:
- joint joint_left_ankle_pitch: limit lower=-0.6 upper=0.6 effort=1000 velocity=10 -> lower=-0.6 upper=0.6 effort=112 velocity=26.1799
- joint joint_left_ankle_roll: limit lower=-0.52 upper=0.52 effort=1000 velocity=10 -> lower=-0.52 upper=0.52 effort=112 velocity=26.1799
- joint joint_left_hip_pitch: limit lower=-1.5 upper=0.3 effort=1000 velocity=10 -> lower=-1.5 upper=0.3 effort=216 velocity=15.1320
- joint joint_left_hip_roll: limit lower=-0.15 upper=0.15 effort=1000 velocity=10 -> lower=-0.15 upper=0.15 effort=216 velocity=15.1320
- joint joint_left_hip_yaw: limit lower=-0.6 upper=0.4 effort=1000 velocity=10 -> lower=-0.6 upper=0.4 effort=112 velocity=26.1799
- joint joint_left_knee_pitch: limit lower=0 upper=2.2 effort=1000 velocity=10 -> lower=0 upper=2.2 effort=216 velocity=15.1320
- joint joint_right_ankle_pitch: limit lower=-0.6 upper=0.6 effort=1000 velocity=10 -> lower=-0.6 upper=0.6 effort=112 velocity=26.1799
- joint joint_right_ankle_roll: limit lower=-0.52 upper=0.52 effort=1000 velocity=10 -> lower=-0.52 upper=0.52 effort=112 velocity=26.1799
- joint joint_right_hip_pitch: limit lower=-1.5 upper=0.3 effort=1000 velocity=10 -> lower=-1.5 upper=0.3 effort=216 velocity=15.1320
- joint joint_right_hip_roll: limit lower=-0.15 upper=0.15 effort=1000 velocity=10 -> lower=-0.15 upper=0.15 effort=216 velocity=15.1320
- joint joint_right_hip_yaw: limit lower=-0.4 upper=0.6 effort=1000 velocity=10 -> lower=-0.4 upper=0.6 effort=112 velocity=26.1799
- joint joint_right_knee_pitch: limit lower=0 upper=2.2 effort=1000 velocity=10 -> lower=0 upper=2.2 effort=216 velocity=15.1320

Commit message: fix(model): align knee limits with calibrated hardware
Set both knee pitch lower limits to -0.1 rad and keep the fixed-base URDF, floating-base URDF, MuJoCo scene, and joint-limit reference table consistent.

File: urdf/export.urdf (robot description, URDF)
Before this commit: robot export, 13 links, 12 joints
Joints:
- joint joint_left_knee_pitch: limit lower=0 upper=2.2 effort=216 velocity=15.1320 -> lower=-0.1 upper=2.2 effort=216 velocity=15.1320
- joint joint_right_knee_pitch: limit lower=0 upper=2.2 effort=216 velocity=15.1320 -> lower=-0.1 upper=2.2 effort=216 velocity=15.1320

File: urdf/export_floating.urdf (robot description, URDF)
Before this commit: robot export_floating, 14 links, 13 joints
Joints:
- joint joint_left_knee_pitch: limit lower=0 upper=2.2 effort=216 velocity=15.1320 -> lower=-0.1 upper=2.2 effort=216 velocity=15.1320
- joint joint_right_knee_pitch: limit lower=0 upper=2.2 effort=216 velocity=15.1320 -> lower=-0.1 upper=2.2 effort=216 velocity=15.1320

Commit message: Update BSRL meshes and collision geometry

File: urdf/export.urdf (robot description, URDF)
Before this commit: robot export, 13 links, 12 joints
Links:
- link base_link: geometry collision box size=0.10 0.10 0.08; collision box size=0.12 0.30 0.035
- link link_left_ankle_pitch: geometry collision cylinder length=0.012 radius=0.025; visual mesh filename=../meshes/link_left_ankle_pitch.obj
- link link_left_ankle_roll: geometry collision cylinder length=0.035 radius=0.025; collision mesh filename=../meshes/left_heel_collision_flat.obj
- link link_left_hip_roll: geometry collision sphere radius=0.04; visual mesh filename=../meshes/link_left_hip_roll.obj
- link link_left_hip_yaw: geometry collision sphere radius=0.04; visual mesh filename=../meshes/link_left_hip_yaw.obj
- link link_left_shank: geometry collision cylinder length=0.2531 radius=0.025; visual mesh filename=../meshes/link_left_shank.obj
- link link_left_thigh: geometry collision cylinder length=0.106 radius=0.035; collision cylinder length=0.16 radius=0.04
- link link_right_ankle_pitch: geometry collision cylinder length=0.012 radius=0.025; visual mesh filename=../meshes/link_right_ankle_pitch.obj
- link link_right_ankle_roll: geometry collision cylinder length=0.035 radius=0.025; collision mesh filename=../meshes/right_heel_collision_flat.obj
- link link_right_hip_roll: geometry collision sphere radius=0.04; visual mesh filename=../meshes/link_right_hip_roll.obj
- link link_right_hip_yaw: geometry collision sphere radius=0.04; visual mesh filename=../meshes/link_right_hip_yaw.obj
- link link_right_shank: geometry collision cylinder length=0.2532 radius=0.025; visual mesh filename=../meshes/link_right_shank.obj
- link link_right_thigh: geometry collision cylinder length=0.106 radius=0.035; collision cylinder length=0.16 radius=0.04
Joints:
- joint joint_left_hip_roll: limit lower=-0.15 upper=0.15 effort=216 velocity=15.1320 -> lower=-0.3 upper=0.3 effort=216 velocity=15.1320
- joint joint_right_hip_roll: limit lower=-0.15 upper=0.15 effort=216 velocity=15.1320 -> lower=-0.3 upper=0.3 effort=216 velocity=15.1320

File: urdf/export_floating.urdf (robot description, URDF)
Before this commit: robot export_floating, 14 links, 13 joints
Links:
- link base_link: geometry collision box size=0.10 0.10 0.08; collision box size=0.12 0.30 0.035
- link link_left_ankle_pitch: geometry collision cylinder length=0.012 radius=0.025; visual mesh filename=../meshes/link_left_ankle_pitch.obj
- link link_left_ankle_roll: geometry collision cylinder length=0.035 radius=0.025; collision mesh filename=../meshes/left_heel_collision_flat.obj
- link link_left_hip_roll: geometry collision sphere radius=0.04; visual mesh filename=../meshes/link_left_hip_roll.obj
- link link_left_hip_yaw: geometry collision sphere radius=0.04; visual mesh filename=../meshes/link_left_hip_yaw.obj
- link link_left_shank: geometry collision cylinder length=0.2531 radius=0.025; visual mesh filename=../meshes/link_left_shank.obj
- link link_left_thigh: geometry collision cylinder length=0.106 radius=0.035; collision cylinder length=0.16 radius=0.04
- link link_right_ankle_pitch: geometry collision cylinder length=0.012 radius=0.025; visual mesh filename=../meshes/link_right_ankle_pitch.obj
- link link_right_ankle_roll: geometry collision cylinder length=0.035 radius=0.025; collision mesh filename=../meshes/right_heel_collision_flat.obj
- link link_right_hip_roll: geometry collision sphere radius=0.04; visual mesh filename=../meshes/link_right_hip_roll.obj
- link link_right_hip_yaw: geometry collision sphere radius=0.04; visual mesh filename=../meshes/link_right_hip_yaw.obj
- link link_right_shank: geometry collision cylinder length=0.2532 radius=0.025; visual mesh filename=../meshes/link_right_shank.obj
- link link_right_thigh: geometry collision cylinder length=0.106 radius=0.035; collision cylinder length=0.16 radius=0.04
Joints:
- joint joint_left_hip_roll: limit lower=-0.15 upper=0.15 effort=216 velocity=15.1320 -> lower=-0.3 upper=0.3 effort=216 velocity=15.1320
- joint joint_right_hip_roll: limit lower=-0.15 upper=0.15 effort=216 velocity=15.1320 -> lower=-0.3 upper=0.3 effort=216 velocity=15.1320
